File: ActiveAeroRP2354.kicad_sch (KiCad schematic)
At the start: 72 parts, among them J1 TAGCONNECT, J2 Conn_01x04_MountingPin, J4 USB_C_Receptacle_USB2.0_16P, Q1 SiA449DJ, Q3 AO3401A, SW1 SW_Push, SW2 SW_Push, U1 RP2354A, U18 AP63205WU, U2 WE-TVS-82400102, U3 W25Q256JVS, U4 ADXL375, U5 MS5611-01BA, U6 SCH16T, U7 BMI563, U9 APS6404L-3SQRx-SN, Y1 ABM8-272-T3

Commit message: basic routing done
Parts:
- added BZ1: Buzzer, Buzzer_Beeper:Buzzer_CUI_CPT-9019S-SMT, symbol Device:Buzzer
- added C26, C27, C28, C29, C31: 1uF, Capacitor_SMD:C_0402_1005Metric, symbol Device:C
- added C30: 10uF, Capacitor_SMD:C_0402_1005Metric, symbol Device:C
- added C43: 10nF, Capacitor_SMD:C_0402_1005Metric, symbol Device:C
- added D6: PPS, LED_SMD:LED_0402_1005Metric, symbol Device:LED
- added FB2: LQG15HS47NJ02, Inductor_SMD:L_0402_1005Metric, symbol Device:FerriteBead
- added J10: UART1_RAD, Connector_JST:JST_GH_SM04B-GHS-TB_1x04-1MP_P1.25mm_Horizontal, symbol Connector_Generic_MountingPin:Conn_01x04_MountingPin
- added J12: SPI, Connector_JST:JST_GH_SM07B-GHS-TB_1x07-1MP_P1.25mm_Horizontal, symbol Connector_Generic_MountingPin:Conn_01x07_MountingPin
- added J3: SRV1, Connector_PinSocket_2.54mm:PinSocket_1x03_P2.54mm_Vertical, symbol Connector_Generic:Conn_01x03
- added J5: UFL, Connector_Coaxial:U.FL_Molex_MCRF_73412-0110_Vertical, symbol Connector:Conn_Coaxial
- added J6: ARM, Connector_JST:JST_XH_B2B-XH-AM_1x02_P2.50mm_Vertical, symbol Connector_Generic:Conn_01x02
- added J7: SRV2, Connector_PinSocket_2.54mm:PinSocket_1x03_P2.54mm_Vertical, symbol Connector_Generic:Conn_01x03
- added J8: SRV4, Connector_PinSocket_2.54mm:PinSocket_1x03_P2.54mm_Vertical, symbol Connector_Generic:Conn_01x03
- added J9: SRV3, Connector_PinSocket_2.54mm:PinSocket_1x03_P2.54mm_Vertical, symbol Connector_Generic:Conn_01x03
- added R16, R17, R18, R7: 220, Resistor_SMD:R_0402_1005Metric, symbol Device:R
- added R54: 10R 0.25W, Resistor_SMD:R_0402_1005Metric, symbol Device:R
- added R56: 1k, Resistor_SMD:R_0402_1005Metric, symbol Device:R
- added U10: AP7347DQ-33W5-7, Package_TO_SOT_SMD:SOT-23-5, symbol Regulator_Linear:AP2112K-1.2
- added U11: MAX-M10S, RF_GPS:ublox_MAX, symbol RF_GPS:MAX-M10S
- added U12: MMC5983MA, Package_LGA:LGA-16_3x3mm_P0.5mm, symbol FCU2025:MMC5983MA
- added U8: AP7347DQ-11W5-7, Package_TO_SOT_SMD:SOT-23-5, symbol Regulator_Linear:AP2112K-1.2
- BATT1: value AMASS_XT30 -> VBAT
- C23: value 10uF -> 22uF
- J1: value TAGCONNECT -> TGCNT
- J2: value Conn_01x04_MountingPin -> I2C
Connections:
- net +1V1: now also C29.1, U8.5 (VOUT)
- net +3V3: now also C27.1, C31.2, J12.2 (Pin_2), U10.5 (VOUT), U11.6 (V_BCKP), U11.7 (VCC_IO), U11.8 (VCC), U12.13 (VDDIO), U12.2 (VDD)
- net +5V: now also C26.1, C28.1, J10.2 (Pin_2), U10.1 (VIN), U10.3 (EN), U8.1 (VIN), U8.3 (EN)
- net +8V4: now also C2.1, C23.1, J3.2 (Pin_2), J7.2 (Pin_2), J8.2 (Pin_2), J9.2 (Pin_2)
- net AC_INT1: now also U1.14 (GPIO10)
- net AC_INT2: now also U1.15 (GPIO11)
- net CS_ACCEL: now also U1.16 (GPIO12)
- net CS_BARO: now also U1.35 (GPIO23)
- net GND: now also BZ1.2 (-), C26.2, C27.2, C28.2, C29.2, C30.1, C31.1, C43.2, J10.1 (Pin_1), J10.MP (MountPin), J12.1 (Pin_1), J12.MP (MountPin), J3.1 (Pin_1), J5.2 (Ext), J7.1 (Pin_1), J8.1 (Pin_1), J9.1 (Pin_1), R56.2, U10.2 (GND), U11.1 (GND), U11.10 (GND), U11.12 (GND), U12.11 (GND), U12.9 (GND), U8.2 (GND)
- net GPIO0: now also U1.2 (GPIO0)
- net IMU1_CS: now also U1.29 (GPIO18)
- net IMU1_INT1: now also U1.28 (GPIO17)
- net IMU_CS: now also U1.36 (GPIO24)
- net IMU_INT: now also U1.41 (GPIO27/ADC1)
- net IMU_RST: now also U1.37 (GPIO25)
- net MISO: now also U1.7 (GPIO4), J12.4 (Pin_4), U12.5 (SDO)
- net MOSI: now also U1.5 (GPIO3), J12.5 (Pin_5), U12.16 (SDA/I)
- net NEOPIX: now also U1.27 (GPIO16)
- net NRST: now also R9.1, U1.26 (RUN), U11.9 (~{RESET})
- net SCK: now also U1.8 (GPIO5), J12.3 (Pin_3), U12.1 (SCL)
- net SCL: now also U1.32 (GPIO20)
- net SDA: now also U1.31 (GPIO19)
- net VBAT: now also J6.2 (Pin_2); no longer C2.1, C23.1, Q1.1 (D)
- net VINSENSE: now also U1.40 (GPIO26/ADC0)
- net SRV_3: now reaches U1.10 (GPIO7)
- net SRV_3: now also R18.2
- net TX2: now reaches U1.12 (GPIO8)
- net TX2: now also U11.3 (RXD)
- net RX2: now reaches U1.13 (GPIO9)
- net RX2: now also U11.2 (TXD)
- net CS_MAG: now reaches U1.17 (GPIO13)
- net CS_MAG: now also U12.4 (~{CS})
- net MAG_INT: now reaches U1.18 (GPIO14)
- net MAG_INT: now also U12.15 (INT)
- net BZ: now reaches U1.19 (GPIO15)
- net BZ: now also BZ1.1 (+)
- net CS1: now reaches U1.3 (GPIO1)
- net CS1: now also J12.6 (Pin_6)
- net TX1: now reaches U1.33 (GPIO21)
- net TX1: now also J10.4 (Pin_4)
- net RX1: now reaches U1.34 (GPIO22)
- net RX1: now also J10.3 (Pin_3)
- net CS2: now reaches U1.4 (GPIO2)
- net CS2: now also J12.7 (Pin_7)
- net SRV_2: now reaches U1.42 (GPIO28/ADC2)
- net SRV_2: now also R16.2
- net SRV_1: now reaches U1.43 (GPIO29/ADC3)
- net SRV_1: now also R7.2
- net SRV_4: now reaches U1.9 (GPIO6)
- net SRV_4: now also R17.2
- new net: J6.1 (Pin_1), Q1.1 (D)
- new net: J9.3 (Pin_3), R18.1
- new net: FB2.1, J5.1 (In), U11.11 (RF_IN)
- new net: C43.1, FB2.2, R54.2
- new net: J7.3 (Pin_3), R16.1
- new net: J8.3 (Pin_3), R17.1
- new net: D6.1 (K), R56.1
- new net: R54.1, U11.14 (VCC_RF)
- new net: D6.2 (A), U11.4 (TIMEPULSE)
- new net: C30.2, U12.10 (CAP)
- new net: J3.3 (Pin_3), R7.1
- new net: U12.12 (NC), U12.14 (NC), U12.3 (NC), U12.6 (NC), U12.7 (NC), U12.8 (NC)
- no-connect marks 7 -> 20
Other:
- note added: "Accel"
- note added: "Baro"
- note added: "Connectors"
- note added: "External IMU"
- note added: "Flash"
- note added: "GPS"
- note added: "Holes"
- note added: "IMU"
- note added: "Indication"
- note added: "Mag"
- note added: "Power"
- note removed: "Add 1v1 and 3v3 LDO"
- note removed: "FLASH"
- moved on the sheet: BATT1, C1, C2, C23, C4, C47, C48, C5, C56, C7, C8, C9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

Commit message: switched to double sided stm32h747xi
Parts:
- removed J12: SPI, Connector_JST:JST_GH_SM07B-GHS-TB_1x07-1MP_P1.25mm_Horizontal, symbol Connector_Generic_MountingPin:Conn_01x07_MountingPin
- removed R11, R15: 27, Resistor_SMD:R_0402_1005Metric, symbol Device:R
- removed R21: 180k, Resistor_SMD:R_0402_1005Metric, symbol Device:R
- removed R22: 56k, Resistor_SMD:R_0402_1005Metric, symbol Device:R
- removed U1: RP2354A, Package_DFN_QFN:QFN-60-1EP_7x7mm_P0.4mm_EP3.4x3.4mm, symbol MCU_RaspberryPi:RP2354A
- removed U11: MAX-M10S, RF_GPS:ublox_MAX, symbol RF_GPS:MAX-M10S
- removed U3: W25Q256JVS, Package_SO:SOIC-8_5.3x5.3mm_P1.27mm, symbol Memory_Flash:W25Q128JVS
- removed U4: ADXL375, Package_LGA:LGA-14_3x5mm_P0.8mm_LayoutBorder1x6y, symbol Sensor_Motion:ADXL343
- removed U8: AP7347DQ-11W5-7, Package_TO_SOT_SMD:SOT-23-5, symbol Regulator_Linear:AP2112K-1.2
- removed Y1: ABM8-272-T3, Crystal:Crystal_SMD_3225-4Pin_3.2x2.5mm, symbol Device:Crystal_GND24_Small
- added C32, C33, C34, C35, C36, C37, C38, C39, C40, C41, C42, C44, C45, C46, C50, C58, C59: 100nF, Capacitor_SMD:C_0402_1005Metric, symbol Device:C
- added C49: 1uF, Capacitor_SMD:C_0402_1005Metric, symbol Device:C
- added C51: 2.2uF, Capacitor_SMD:C_0402_1005Metric, symbol Device:C
- added C52, C53: 4.7uF, Capacitor_SMD:C_0402_1005Metric, symbol Device:C
- added C54, C55: 10uF, Capacitor_SMD:C_0402_1005Metric, symbol Device:C
- added C57: 220pF, Capacitor_SMD:C_0402_1005Metric, symbol Device:C
- added FB1: FCM1608KF-601T03, Inductor_SMD:L_0402_1005Metric, symbol Device:FerriteBead_Small
- added FB3: LSMCA160808T180NGR, Inductor_SMD:L_0603_1608Metric, symbol Device:FerriteBead_Small
- added J11: SPI, Connector_JST:JST_GH_SM08B-GHS-TB_1x08-1MP_P1.25mm_Horizontal, symbol Connector_Generic_MountingPin:Conn_01x08_MountingPin
- added J12: UART3, Connector_JST:JST_GH_SM04B-GHS-TB_1x04-1MP_P1.25mm_Horizontal, symbol Connector_Generic_MountingPin:Conn_01x04_MountingPin
- added J13: RUNCAM, Connector_JST:JST_GH_SM04B-GHS-TB_1x04-1MP_P1.25mm_Horizontal, symbol Connector_Generic_MountingPin:Conn_01x04_MountingPin
- added L1: L_Small, Inductor_SMD:L_Changjiang_FTC201607S, symbol Device:L_Small
- added R19, R23, R25: 10k, Resistor_SMD:R_0402_1005Metric, symbol Device:R
- added R20: 51, Resistor_SMD:R_0402_1005Metric, symbol Device:R
- added U1: LSM6DSV320, Package_LGA:LGA-14_3x2.5mm_P0.5mm_LayoutBorder3x4y, symbol Sensor_Motion:LSM6DS3
- added U13: STM32H747XIHx, Package_BGA:TFBGA-265_14x14mm_Layout17x17_P0.8mm, symbol MCU_ST_STM32H7:STM32H747XIHx
- added U3: MIA-M10Q, Package_LGA:ublox_LGA-53_4.5x4.5mm_Layout9x9_P0.5mm, symbol RF_GPS:MIA-M10Q
- added U4: W25N512GV, Package_SON:WSON-8-1EP_6x5mm_P1.27mm_EP3.4x4.3mm, symbol Memory_Flash:W25Q128JVP
- added U8: INA238, Package_SO:VSSOP-10_3x3mm_P0.5mm, symbol Sensor_Energy:INA238
- added Y1: ECS-.327-6-1210-TR, Crystal:Crystal_SMD_MicroCrystal_CM9V-T1A-2Pin_1.6x1.0mm, symbol Device:Crystal
- added Y2: 32.768khz, Crystal:Crystal_SMD_MicroCrystal_CM9V-T1A-2Pin_1.6x1.0mm, symbol Device:Crystal
- added Y3: 25Mhz, Oscillator:Oscillator_SMD_Abracon_ASCO-4Pin_1.6x1.2mm, symbol Oscillator:ASCO
- C10, C11: value 15pF -> 100nF
- C19: value 10uF -> 100nF
- C22, C25: value 4.7uF -> 1uF
- C28, C29: value 1uF -> 8pF
- C7: value 0.1uF -> 100nF
- C8: value 1uF -> 100nF
- J6: footprint Connector_JST:JST_XH_B2B-XH-AM_1x02_P2.50mm_Vertical -> Connector_JST:JST_PH_B2B-PH-K_1x02_P2.00mm_Vertical
- R10: value 1k -> 10k
- R9: value 1k -> 0.01R; footprint Resistor_SMD:R_0402_1005Metric -> Resistor_SMD:R_2512_6332Metric
Connections:
- net +3V3: now also C10.1, C11.1, R10.2, R4.2, C32.1, C33.1, C34.1, C35.1, C36.1, C37.1, C38.1, C39.1, C40.1, C41.1, C42.1, C44.1, C45.1, C46.1, C49.1, C59.1, FB1.1, FB3.1, J11.2 (Pin_2), J12.2 (Pin_2), R19.1, U1.5 (VDDIO), U1.8 (VDD), U13.B1 (VBAT), U13.E11 (VDD), U13.E6 (VDD), U13.E9 (VDD), U13.F17 (VDD33_USB), U13.F5 (VDD), U13.G13 (VDD), U13.G17 (VDD50_USB), U13.G5 (VDD), U13.H13 (VDD), U13.H5 (VDD), U13.J13 (VDD), U13.K13 (VDD), U13.K5 (VDD), U13.L13 (VDD), U13.L5 (VDD), U13.M13 (VDD), U13.M5 (VDD), U13.N10 (VDD), U13.N11 (VDD), U13.N12 (VDD), U13.N7 (VDD), U13.N8 (VDD), U13.P17 (VDDDSI), U3.B1 (VCC), U3.J4 (V_IO), U3.J5 (V_BCKP), U4.8 (VCC), U8.6 (VS), Y3.4 (VDD); no longer R4.1
- net +5V: no longer C28.1
- net +8V4: now also J11.8 (Pin_8), U8.8 (Vbus)
- net AC_INT1: now also U1.4 (INT1), U13.N4 (PA1)
- net AC_INT2: now also U1.9 (INT2), U13.N2 (PH2)
- net BZ: now also U13.A16 (PI0)
- net CS1: now also J11.6 (Pin_6), U13.D16 (PH13)
- net CS2: now also J11.7 (Pin_7), U13.B17 (PH14)
- net CS_ACCEL: now also R19.2, U1.12 (CS), U13.P2 (PH3); no longer R4.2
- net CS_BARO: now also U13.F4 (PI11)
- net CS_MAG: now also U13.U2 (PA3)
- net GND: now also C10.2, C11.2, C20.2, R9.1, C32.2, C33.2, C34.2, C35.2, C36.2, C37.2, C38.2, C39.2, C40.2, C41.2, C42.2, C44.2, C45.2, C46.2, C49.2, C50.2, C51.2, C52.2, C53.2, C54.2, C55.1, C57.2, C58.2, C59.2, J11.1 (Pin_1), J11.MP (MountPin), J12.1 (Pin_1), J12.MP (MountPin), J13.1 (Pin_1), J13.MP (MountPin), R25.2, U1.6 (GND), U1.7 (GND), U13.A1 (VSS), U13.A17 (VSS), U13.B2 (VSS), U13.B6 (VSS), U13.C10 (VSS), U13.C13 (VSS), U13.C16 (VSS), U13.F2 (VSSSMPS), U13.G10 (VSS), U13.G11 (VSS), U13.G16 (VSS), U13.G7 (VSS), U13.G8 (VSS), U13.G9 (VSS), U13.H10 (VSS), U13.H11 (VSS), U13.H7 (VSS), U13.H8 (VSS), U13.H9 (VSS), U13.J10 (VSS), U13.J11 (VSS), U13.J16 (VSS), U13.J17 (VSS), U13.J3 (VSS), U13.J7 (VSS), U13.J8 (VSS), U13.J9 (VSS), U13.K10 (VSS), U13.K11 (VSS), U13.K15 (VSSDSI), U13.K7 (VSS), U13.K8 (VSS), U13.K9 (VSS), U13.L10 (VSS), U13.L11 (VSS), U13.L15 (VSSDSI), U13.L7 (VSS), U13.L8 (VSS), U13.L9 (VSS), U13.M15 (VSSDSI), U13.N1 (VREF-), U13.N16 (VSS), U13.P1 (VSSA), U13.R4 (VSS), U13.R8 (VSS), U13.T12 (VSS), U13.U1 (VSS), U13.U17 (VSS), U3.A1 (GND), U3.A2 (GND), U3.A3 (GND), U3.A8 (GND), U3.A9 (GND), U3.B2 (GND), U3.B8 (GND), U3.C3 (GND), U3.C9 (GND), U3.E3 (GND), U3.E4 (GND), U3.E9 (GND), U3.F1 (GND), U3.F3 (GND), U3.F4 (GND), U3.F9 (Reserved), U3.G3 (GND), U3.G4 (GND), U3.G5 (GND), U3.G6 (GND), U3.G7 (Reserved), U3.H8 (GND), U3.J8 (GND), U3.J9 (GND), U4.4 (GND), U4.9 (EP), U8.1 (A1), U8.10 (Vin+), U8.2 (A0), U8.7 (GND), Y3.2 (GND); no longer BATT1.1 (Pin_1), C10.1, C11.1, C20.1
- net IMU1_CS: now also U13.M2 (PC1)
- net IMU1_INT1: now also U13.H4 (PF3)
- net IMU1_INT2: now also U13.G4 (PF0)
- net IMU_CS: now also U13.C4 (PE0)
- net IMU_INT: now also U13.A4 (PI4)
- net IMU_RST: now also U13.D3 (PE3)
- net MAG_INT: now also U13.U4 (PC5)
- net MISO: now also U1.1 (SDO/SA0), U13.D1 (PE5)
- net MOSI: now also U1.14 (SDA), U13.E5 (PE6)
- net NEOPIX: now also U13.U5 (PB0)
- net NRST: now also SW2.1, C58.1, U13.K1 (NRST), U3.C4 (~{RESET}); no longer R9.1
- net QSPI_SCK: now also U13.L3 (PF10), U4.6 (CLK)
- net RX1: now also U13.T15 (PB15)
- net RX2: now also U13.E2 (PI9), U3.G1 (TX)
- net SCK: now also U1.13 (SCL), U13.C3 (PE2)
- net SCL: now also U13.R16 (PD12), U8.4 (SDA)
- net SDA: now also U13.R17 (PD13), U8.5 (SCL)
- net SRV_1: now also U13.A3 (PI5)
- net SRV_2: now also U13.A2 (PI6)
- net SRV_3: now also U13.B3 (PI7)
- net SRV_4: now also U13.E14 (PC9)
- net SWCLK: now also U13.B14 (PA14)
- net SWDIO: now also U13.C15 (PA13)
- net TX1: now also U13.U15 (PB14)
- net TX2: now also U13.D4 (PB9), U3.H1 (RX)
- net USB_D+: now also U2.4, U13.E16 (PA12)
- net USB_D-: now also U2.6, U13.E17 (PA11)
- net VBUS: now also R23.1
- net at R10.1: now also Y3.1 (Tri-State)
- net at FB2.1, J5.1 (In): now also U3.B9 (RF_IN)
- net SWO: now reaches J1.6 (SWO)
- net SWO: now also U13.C6 (PB3)
- net at R54.1: now also U3.C6 (VCC_RF)
- net at D6.2 (A): now also U3.A7 (TIMEPULSE)
- net MON_GND: now reaches R9.2
- net MON_GND: now also BATT1.1 (Pin_1), U8.9 (Vin-); no longer SW2.1
- net +1V1 renamed VDDA
- net VDDA: now also C20.1, FB1.2, U13.L1 (VDDA), U13.M1 (VREF+); no longer C20.2, C29.1
- net GPIO0 renamed PSRAM_CS
- net PSRAM_CS: now also U13.B13 (PC11)
- net QSPI_SD0 renamed PSRAM_SD0
- net PSRAM_SD0: now also U13.U9 (PE7)
- net QSPI_SD1 renamed PSRAM_SD1
- net PSRAM_SD1: now also U13.T9 (PE8)
- net QSPI_SD2 renamed PSRAM_SD2
- net PSRAM_SD2: now also U13.P9 (PE9)
- net QSPI_SD3 renamed PSRAM_SD3
- net PSRAM_SD3: now also U13.N9 (PE10)
- net QSPI_SS: no longer names the net of R8.1
- net QSPI_SS: now also U13.E8 (BOOT0); no longer R3.2
- new net: R4.1, U13.E7 (PDR_ON)
- new net: U3.A5 (RTC_O), Y2.1
- new net: U3.A4 (RTC_I), Y2.2
- new net: C29.1, U13.C1 (PC15), Y1.1
- new net: C55.2, FB3.2, U13.F1 (VDDSMPS)
- new net: R20.2, Y3.3 (OUT)
- new net: C50.1, C51.1, U13.N17 (VCAPDSI)
- new net: C28.1, U13.C2 (PC14), Y1.2
- new net FLASH_CS: R3.2, U13.P11 (PB10), U4.1 (~{CS})
- new net FLASH_SD0: U13.K4 (PF8), U4.5 (DI/IO_{0})
- new net FLASH_SD1: U13.L4 (PF9), U4.2 (DO/IO_{1})
- new net FLASH_SD2: U13.K3 (PF7), U4.3 (~{WP}/IO_{2})
- new net FLASH_SD3: U13.K2 (PF6), U4.7 (~{HOLD}/~{RESET}/IO_{3})
- new net MISO1: J11.4 (Pin_4), U13.B15 (PI2)
- new net MOSI1: J11.5 (Pin_5), U13.C14 (PI3)
- new net OSC_IN: R20.1, U13.J2 (PH0)
- new net PA9: R23.2, R25.1, U13.D15 (PA9)
- new net RX3: J12.3 (Pin_3), U13.A5 (PB5)
- new net RX4: J13.3 (Pin_3), U13.B11 (PD6)
- new net SCK1: J11.3 (Pin_3), U13.A15 (PI1)
- new net TX3: J12.4 (Pin_4), U13.B5 (PB6)
- new net TX4: J13.4 (Pin_4), U13.A11 (PD5)
- new net VDDSDC: C52.1, C53.1, C54.1, L1.1, U13.A6 (VDDLDO), U13.A7 (VCAP), U13.C17 (VDDLDO), U13.D17 (VCAP), U13.G2 (VFBSMPS), U13.U11 (VCAP), U13.U12 (VDDLDO)
- new net VLXSMPS: C57.1, L1.2, U13.E1 (VLXSMPS)
- no-connect marks 20 -> 23
Other:
- moved on the sheet: C12, C13, C14, C15, C16, C17, C18, C24, C26, C27, C43, C7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

Commit message: design lock (probably), added silks
Parts:
- added C60, C61: 100nF, Capacitor_SMD:C_0402_1005Metric, symbol Device:C
- added C62: 4.7uF, Capacitor_SMD:C_0402_1005Metric, symbol Device:C
- added C63, C64: 100pF, Capacitor_SMD:C_0402_1005Metric, symbol Device:C
- added D4: ESD2CANFD24, Package_TO_SOT_SMD:SOT-23-3, symbol Power_Protection:ESDA5V3L
- added J14: Conn_01x06_MountingPin, Connector_JST:JST_GH_SM06B-GHS-TB_1x06-1MP_P1.25mm_Horizontal, symbol Connector_Generic_MountingPin:Conn_01x06_MountingPin
- added J15: Conn_01x03_MountingPin, Connector_JST:JST_GH_SM03B-GHS-TB_1x03-1MP_P1.25mm_Horizontal, symbol Connector_Generic_MountingPin:Conn_01x03_MountingPin
- added L2: DLW32SH101XF2L, FCU2025Lib:FIL_DLW32SH101XF2L, symbol Device:L_Ferrite_Coupled_1243
- added Q2: AO3401A, Package_TO_SOT_SMD:SOT-23, symbol Transistor_FET:AO3401A
- added R11: 220, Resistor_SMD:R_0402_1005Metric, symbol Device:R
- added R15, R21, R22: 10k, Resistor_SMD:R_0402_1005Metric, symbol Device:R
- added R26, R27: 60R, Resistor_SMD:R_0402_1005Metric, symbol Device:R
- added U11: MCP2562-E-MF, Package_DFN_QFN:DFN-8-1EP_3x3mm_P0.65mm_EP1.55x2.4mm, symbol Interface_CAN_LIN:MCP2562-E-MF
Connections:
- net +3V3: now also C61.2, R15.2, R21.1, R22.1, U11.5 (Vio)
- net +5V: now also C60.1, J14.1 (Pin_1), U11.3 (VDD)
- net +8V4: now also Q2.2 (S)
- net GND: now also C60.2, C61.1, C62.2, C63.2, C64.1, D4.3 (A), J14.6 (Pin_6), J14.MP (MountPin), J15.2 (Pin_2), J15.MP (MountPin), U11.2 (VSS), U11.9 (PAD)
- net NRST: no longer U3.C4 (~{RESET})
- net SCL: no longer J2.4 (Pin_4)
- net SDA: no longer J2.3 (Pin_3)
- net ALRT: now reaches U8.3 (~{Alert})
- net ALRT: now also U13.P16 (PD14)
- net at J13.2 (Pin_2): now also Q2.3 (D)
- net GPS_INT: now reaches U3.A6 (EXTINT)
- net GPS_INT: now also U13.C11 (PD7)
- net RX5: now reaches U13.A10 (PG9)
- net RX5: now also J14.3 (Pin_3)
- net CAM_SW: now reaches U13.A14 (PA15)
- net CAM_SW: now also R11.2, R15.1
- net GPS_RST: now reaches U13.B10 (PJ15)
- net GPS_RST: now also U3.C4 (~{RESET})
- net RTS5: now reaches U13.C9 (PG12)
- net RTS5: now also J14.5 (Pin_5)
- net TX5: now reaches U13.D6 (PG15)
- net TX5: now also J14.2 (Pin_2)
- net CTS5: now reaches U13.D8 (PG14)
- net CTS5: now also J14.4 (Pin_4)
- net CAN_SHDN: now reaches U13.P5 (PI15)
- net CAN_SHDN: now also U11.8 (SHDN)
- net SDA1: now reaches U13.T13 (PH8)
- net SDA1: now also J2.3 (Pin_3), R21.2
- net CAN_RX: now reaches U13.T14 (PB12)
- net CAN_RX: now also U11.4 (RXD)
- net SCL1: now reaches U13.U13 (PH7)
- net SCL1: now also J2.4 (Pin_4), R22.2
- net CAN_TX: now reaches U13.U14 (PB13)
- net CAN_TX: now also U11.1 (TXD)
- new net: Q2.1 (G), R11.1
- new net: C64.2, D4.2 (K), J15.3 (Pin_3), L2.2, R27.2
- new net: C63.1, D4.1 (K), J15.1 (Pin_1), L2.3, R26.1
- new net: C62.1, R26.2, R27.1
- new net: L2.1, U11.6 (CANL)
- new net: L2.4, U11.7 (CANH)
- no-connect marks 23 -> 28
Other:
- moved on the sheet: J13

Commit message: cleaned up silkscreens and layout
Other:
- note added: "BATTERY"
- note added: "CAN"
- note added: "POWER MONITOR"
- note added: "SERVO"
- note removed: "I2C"
- moved on the sheet: BATT1, BZ1, C10, C11, C12, C13, C14, C15, C16, C17, C18, C19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

Commit message: finished silks
Parts:
- added C65, C66: 100nF, Capacitor_SMD:C_0402_1005Metric, symbol Device:C
Connections:
- net +5V: now also C65.2, C66.2
- net GND: now also C65.1, C66.1
